Commit message: Move-it werkt eindelijk weer

File: my_ufactory_ROS2/my_uf_description/urdf/uf_robot.urdf.xacro (robot description, xacro)
@@ -6,5 +6,5 @@
   <xacro:arg name="effort_control" default="false"/>
   <xacro:arg name="velocity_control" default="false"/>
-  <xacro:arg name="add_gripper" default="false"/>
+  <xacro:arg name="add_gripper" default="true"/>
   <xacro:arg name="add_vacuum_gripper" default="false"/>
   <xacro:arg name="model1300" default="false"/>
@@ -167,6 +167,5 @@
     <material>Gazebo/Red</material>
   </gazebo>
-  <!-- tool center point -->
-<!--
+    <!-- tool center point -->
   <link name="tcp_link" />
   <joint name="tool_link" type="fixed">
@@ -174,4 +173,32 @@
     <child link="tcp_link" />
     <origin xyz="0.0 0.0 0.0" rpy="0.0 0.0 0.0"/>
+  </joint>
+  <!-- Gripper Lite6 -->
+<!--
+  <link name="gripper_lite6_link">
+    <visual>
+      <origin xyz="0 0 0" rpy="0 0 0"/>
+      <geometry>
+        <mesh filename="package://my_uf_description/meshes/Gripper_Lite.stl" scale="1 1 1"/>
+      </geometry>
+      <material name="gray">
+        <color rgba="0.6 0.6 0.6 1.0"/>
+      </material>
+    </visual>
+    <collision>
+      <origin xyz="0 0 0" rpy="0 0 0"/>
+      <geometry>
+        <mesh filename="package://my_uf_description/meshes/Gripper_Lite.stl" scale="1 1 1"/>
+      </geometry>
+    </collision>
+    <inertial>
+      <mass value="2.0"/>
+      <inertia ixx="1.0" ixy="1.0" ixz="1.0" iyy="1.0" iyz="1.0" izz="1.0"/>
+    </inertial>
+  </link>
+  <joint name="gripper_lite6_joint" type="fixed">
+    <parent link="tcp_link"/>
+    <child link="gripper_lite6_link"/>
+    <origin xyz="-0.105 -0.03875 -0.02" rpy="0 0 0"/>
   </joint>
 -->

File: my_ufactory_ROS2/my_uf_moveit_config/config/uf_robot.urdf.xacro (robot description, xacro)
@@ -1,13 +1,5 @@
 <?xml version="1.0"?>
 <robot xmlns:xacro="http://www.ros.org/wiki/xacro" name="uf_robot">
-    <xacro:arg name="initial_positions_file" default="initial_positions.yaml" />
-    <xacro:arg name="add_gripper" default="true"/>
-    <xacro:arg name="add_vacuum_gripper" default="false"/>
     <!-- Import uf_robot urdf file -->
     <xacro:include filename="$(find my_uf_description)/urdf/uf_robot.urdf.xacro" />
-    <!-- Import control_xacro -->
-    <xacro:include filename="uf_robot.ros2_control.xacro" />
-    <!--
-    <xacro:uf_robot_ros2_control name="FakeSystem" initial_positions_file="$(arg initial_positions_file)"/>
-    -->
 </robot>

Commit message: Gripper met draad

File: my_ufactory_ROS2/my_uf_description/urdf/uf_robot.urdf.xacro (robot description, xacro)
@@ -175,10 +175,9 @@
   </joint>
   <!-- Gripper Lite6 -->
-<!--
   <link name="gripper_lite6_link">
     <visual>
       <origin xyz="0 0 0" rpy="0 0 0"/>
       <geometry>
-        <mesh filename="package://my_uf_description/meshes/Gripper_Lite.stl" scale="1 1 1"/>
+        <mesh filename="package://my_uf_description/meshes/Gripper_Lite.STL" scale="1 1 1"/>
       </geometry>
       <material name="gray">
@@ -189,5 +188,5 @@
       <origin xyz="0 0 0" rpy="0 0 0"/>
       <geometry>
-        <mesh filename="package://my_uf_description/meshes/Gripper_Lite.stl" scale="1 1 1"/>
+        <mesh filename="package://my_uf_description/meshes/Gripper_Lite.STL" scale="1 1 1"/>
       </geometry>
     </collision>
@@ -202,5 +201,4 @@
     <origin xyz="-0.105 -0.03875 -0.02" rpy="0 0 0"/>
   </joint>
--->
     <gazebo reference="world">
       <turnGravityOff>true</turnGravityOff>

Commit message: Verbetering zodat hij niet in collision staat bij oppakken

File: my_ufactory_ROS2/my_uf_description/urdf/uf_robot.urdf.xacro (robot description, xacro)
@@ -121,5 +121,5 @@
       <origin xyz="0 0 0.0" />
       <geometry>
-        <box size="0.7 1.1 0.03" />
+        <box size="0.6 0.8 0.02" />
       </geometry>
     </collision>

Commit message: Voorwerp in gripper geplaatst

File: my_ufactory_ROS2/my_uf_description/urdf/uf_robot.urdf.xacro (robot description, xacro)
@@ -204,4 +204,34 @@
       <turnGravityOff>true</turnGravityOff>
     </gazebo>
+  <!--object zodat hij niet tegen tussenwand aankomt-->
+  <link name="held_object_link">
+    <visual>
+      <origin xyz="0 0 0" rpy="0 0 0"/>
+      <geometry>
+        <box size="0.078 0.0403 0.0624"/>
+      </geometry>
+      <material name="held_object_debug">
+        <color rgba="1 0 1 0.4"/>
+      </material>
+    </visual>
+    <collision>
+      <origin xyz="0 0 0" rpy="0 0 0"/>
+      <geometry>
+        <box size="0.08 0.045 0.07"/>
+      </geometry>
+    </collision>
+    <inertial>
+      <origin xyz="0 0 0" rpy="0 0 0"/>
+      <mass value="0.1"/>
+      <inertia ixx="0.0001" ixy="0" ixz="0"
+              iyy="0.0001" iyz="0"
+              izz="0.0001"/>
+    </inertial>
+  </link>
+  <joint name="held_object_joint" type="fixed">
+    <parent link="uflite_gripper_link"/>
+    <child link="held_object_link"/>
+    <origin xyz="0 0 0.1" rpy="0 0 0"/>
+  </joint>
   <!--Door mij toegevoegd-->
   <xacro:include filename="$(find my_uf_description)/urdf/assembly.urdf.xacro"/>

Commit message: Ja

File: my_ufactory_ROS2/my_uf_description/urdf/uf_robot.urdf.xacro (robot description, xacro)
@@ -6,5 +6,5 @@
   <xacro:arg name="effort_control" default="false"/>
   <xacro:arg name="velocity_control" default="false"/>
-  <xacro:arg name="add_gripper" default="true"/>
+  <xacro:arg name="add_gripper" default="false"/>
   <xacro:arg name="add_vacuum_gripper" default="false"/>
   <xacro:arg name="model1300" default="false"/>
@@ -205,4 +205,5 @@
     </gazebo>
   <!--object zodat hij niet tegen tussenwand aankomt-->
+<!-- object zodat hij niet tegen tussenwand aankomt -->
   <link name="held_object_link">
     <visual>
@@ -230,5 +231,5 @@
   </link>
   <joint name="held_object_joint" type="fixed">
-    <parent link="uflite_gripper_link"/>
+    <parent link="link6"/>
     <child link="held_object_link"/>
     <origin xyz="0 0 0.1" rpy="0 0 0"/>

Commit message: Werkt soortvan

File: my_ufactory_ROS2/my_uf_description/urdf/uf_robot.urdf.xacro (robot description, xacro)
@@ -219,5 +219,5 @@
       <origin xyz="0 0 0" rpy="0 0 0"/>
       <geometry>
-        <box size="0.08 0.045 0.07"/>
+        <box size="0.07 0.0403 0.0624"/>
       </geometry>
     </collision>
